File: hardware/Berker Integro sensor/wemos-multi-carrier/berker-sensor.kicad_pcb (KiCad board)
At the start: 2 copper layers, 41 x 41 mm, 4 parts, among them J1 Conn_01x02, J3 Conn_01x08_Male, J4 Conn_01x08_Male, U1 WeMos_mini

Commit message: Tweak
Parts:
- added J2: USB_B_Micro, Connector_USB:USB_Micro-B_Wuerth_614105150721_Vertical, F.Cu at (-1.30, 13.8)
- added K1: Relay_DPDT, pdjr:RS_SUBMINIATURE_SIGNAL_RELAY, F.Cu at (5.00, -1.10)
- added K2: Relay_DPDT, pdjr:RS_SUBMINIATURE_SIGNAL_RELAY, F.Cu at (-5.00, -1.10)
- added Q1: 2N7002, Package_TO_SOT_SMD:SOT-23, F.Cu at (2.83, 2.50)
- added Q3: 2N7002, Package_TO_SOT_SMD:SOT-23, F.Cu at (-7.17, 2.50)
- added R1: 4K8, Resistor_SMD:R_0805_2012Metric, F.Cu at (16.1, 5.65)
- added R2: 4K8, Resistor_SMD:R_0805_2012Metric, F.Cu at (16.1, 3.15)
- added R3: 10K, Resistor_SMD:R_0805_2012Metric, F.Cu at (6.66, 2.50)
- added R5: 10K, Resistor_SMD:R_0805_2012Metric, F.Cu at (-3.45, 2.50)
- J1: value Conn_01x02 -> Conn_01x04_Socket; footprint Connector_PinHeader_2.54mm:PinHeader_1x02_P2.54mm_Vertical -> Connector_JST:JST_GH_SM04B-GHS-TB_1x04-1MP_P1.25mm_Horizontal; moved to B.Cu
- J3, J4: value Conn_01x08_Male -> Screw_Terminal_01x03; footprint TerminalBlock_Phoenix:TerminalBlock_Phoenix_MPT-0,5-8-2.54_1x08_P2.54mm_Horizontal -> pdjr:RS_1731204_2.54x3_SCREW_TERMINAL
- moved J1 25.4 mm to (0.00, 7.03), turned to 0 degrees
- moved J3 8.01 mm to (-4.40, -15.3), turned to 0 degrees
- moved J4 8.01 mm to (4.40, -15.3), turned to 0 degrees
Connections:
- J1 pad 1: +3V3 -> Net-(J1-Pin_1)
- J1 pad 2: GND -> Net-(J1-Pin_2)
- J3 pad 1: +3V3 -> Net-(J3-Pin_1)
- J3 pad 2: Net-(J3-Pad2) -> Net-(J3-Pin_2)
- J3 pad 3: Net-(J3-Pad3) -> Net-(J3-Pin_3)
- J4 pad 1: Net-(J4-Pad1) -> Net-(J4-Pin_1)
- J4 pad 2: GND -> Net-(J4-Pin_2)
- J4 pad 3: Net-(J4-Pad3) -> Net-(J4-Pin_3)
- U1 pad 1: Net-(J4-Pad1) -> +5V
- U1 pad 10: Net-(J3-Pad7) -> unconnected-(U1-A0-Pad10)
- U1 pad 11: Net-(J3-Pad6) -> unconnected-(U1-D0-Pad11)
- U1 pad 12: Net-(J3-Pad5) -> unconnected-(U1-D5-Pad12)
- U1 pad 13: Net-(J3-Pad4) -> unconnected-(U1-D6-Pad13)
- U1 pad 14: Net-(J3-Pad3) -> unconnected-(U1-D7-Pad14)
- U1 pad 15: Net-(J3-Pad2) -> unconnected-(U1-D8-Pad15)
- U1 pad 3: Net-(J4-Pad3) -> /R1
- U1 pad 4: Net-(J4-Pad4) -> /R0
- U1 pad 5: Net-(J4-Pad5) -> Net-(J1-Pin_2)
- U1 pad 6: Net-(J4-Pad6) -> Net-(J1-Pin_1)
- U1 pad 7: Net-(J4-Pad7) -> unconnected-(U1-Rx-Pad7)
- U1 pad 8: Net-(J4-Pad8) -> unconnected-(U1-Tx-Pad8)
- U1 pad 9: Net-(J3-Pad8) -> unconnected-(U1-Rst-Pad9)
Routing:
- net +5V: track 0.00 -> 53.7 mm, vias 0 -> 3
- net +3V3: track 24.2 -> 1.76 mm, vias 0 -> 1
- net Net-(J1-Pin_2): track 0.00 -> 20.6 mm, vias 0 -> 1
- net Net-(J1-Pin_1): track 0.00 -> 20.0 mm, vias 0 -> 1
- net /R1: track 0.00 -> 18.4 mm
- net Net-(J3-Pin_3): track 0.00 -> 18.2 mm, vias 0 -> 1
- net Net-(J4-Pin_1): track 0.00 -> 18.1 mm, vias 0 -> 1
- net GND: track 21.6 -> 4.36 mm, vias 0 -> 2
- net Net-(J4-Pin_2): track 0.00 -> 15.9 mm, vias 0 -> 1
- net Net-(J3-Pin_2): track 0.00 -> 15.8 mm, vias 0 -> 1
- net Net-(J4-Pin_3): track 0.00 -> 13.5 mm
- net Net-(J3-Pin_1): track 0.00 -> 13.5 mm
- net /R0: track 0.00 -> 4.91 mm
- net Net-(J4-Pad1): track 4.87 -> 0.00 mm
- net Net-(J3-Pad2): track 4.84 -> 0.00 mm
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- added copper zone on F.Cu, net +3V3
- removed copper zone on F.Cu, net GND
Other:
- outline, holes or cut-outs redrawn
- net class Default removed
- net class Mains removed
- board text added: "2024 (c) Paul Reeve <preeve@pdjr.eu>"
- board text removed: "3V3"
- board text removed: "D1"
- board text removed: "D2"
- board text removed: "https://github.com/pdjr-wemos/MULTI001 2024 (c) Paul Reeve preeve@pdjr.eu"
