File: hardware/multi001-v1/multi001-v1.kicad_pcb (KiCad board)
At the start: 2 copper layers, 26 parts, among them J1 Screw_Terminal_01x02, J2 Screw_Terminal_01x04, J3 Screw_Terminal_01x03, J4 Screw_Terminal_01x02, J5 Screw_Terminal_01x02, J6 Screw_Terminal_01x02, J7 Screw_Terminal_01x02, J8 Screw_Terminal_01x04, SW1 SW_SPST, SW2 SW_SPST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

Commit message: Tweak
Parts:
- removed C1 (x2): 10uF, Capacitor_THT:CP_Radial_D6.3mm_P2.50mm
- removed C2: CP, Capacitor_THT:CP_Radial_D8.0mm_P3.80mm
- removed C2: 22uF, Capacitor_THT:CP_Radial_D6.3mm_P2.50mm
- removed F1: Fuse, Fuse:Fuseholder_Cylinder-5x20mm_Bulgin_FX0456_Vertical_Closed
- removed J2: Screw_Terminal_01x04, Connector_PinHeader_2.54mm:PinHeader_1x04_P2.54mm_Vertical
- removed J3: Screw_Terminal_01x03, Connector_PinHeader_2.54mm:PinHeader_1x03_P2.54mm_Vertical
- removed J4, J5, J6, J7: Screw_Terminal_01x02, Connector_PinHeader_2.54mm:PinHeader_1x02_P2.54mm_Vertical
- removed R3: 9K1, Resistor_THT:R_Axial_DIN0207_L6.3mm_D2.5mm_P7.62mm_Horizontal
- removed R5: 4K7, Resistor_THT:R_Axial_DIN0207_L6.3mm_D2.5mm_P7.62mm_Horizontal
- removed SW1, SW2, SW3, SW4: SW_SPST, Connector_PinHeader_2.54mm:PinHeader_1x02_P2.54mm_Vertical
- removed U2: VTX-214-001-103, transformers:VTX214001103
- removed U2: DS18B20, Package_TO_SOT_THT:TO-92_Inline
- added K1: SANYOU_SRD_Form_A, Relay_THT:Relay_SPST_SANYOU_SRD_Series_Form_A, F.Cu at (51.0, 89.2)
- added Q1: 2N7002, Package_TO_SOT_SMD:SOT-23, F.Cu at (28.5, 125.1)
- J1 (x2): footprint Connector_PinHeader_2.54mm:PinHeader_1x02_P2.54mm_Vertical -> Connector_PinHeader_2.00mm:PinHeader_1x02_P2.00mm_Vertical_SMD_Pin1Right
- R1: value 3K2 -> 100K; footprint Resistor_THT:R_Axial_DIN0207_L6.3mm_D2.5mm_P7.62mm_Horizontal -> Resistor_SMD:R_0805_2012Metric
- R2: value 9K1 -> 4K8; footprint Resistor_THT:R_Axial_DIN0207_L6.3mm_D2.5mm_P7.62mm_Horizontal -> Resistor_SMD:R_0805_2012Metric
- R4: value 3K2 -> 4K8; footprint Resistor_THT:R_Axial_DIN0207_L6.3mm_D2.5mm_P7.62mm_Horizontal -> Resistor_SMD:R_0805_2012Metric
- moved J8 130.7 mm to (47.1, 109.7), turned to 90 degrees
Connections:
- J1 pad 1: +12V -> Net-(J1-Pin_1)
- J1 pad 2: GND -> Net-(J1-Pin_2)
- J1 pad 1: Net-(F1-Pad2) -> Net-(J1-Pin_1)
- J1 pad 2: Net-(C1-Pad2) -> Net-(J1-Pin_2)
- R1 pad 1: GND -> /RELAY
- R1 pad 2: /PIR -> Net-(Q1-G)
- R2 pad 1: /PIR -> /SDA
- R2 pad 2: Net-(J2-Pad2) -> +3V3
- R4 pad 1: /LUX -> /SCL
- R4 pad 2: GND -> +3V3
- U1 pad 1: Net-(U1-Pad1) -> +5V
- U1 pad 10: /LUX -> unconnected-(U1-A0-Pad10)
- U1 pad 11: /PIR -> unconnected-(U1-D0-Pad11)
- U1 pad 12: Net-(U1-Pad12) -> unconnected-(U1-D5-Pad12)
- U1 pad 13: Net-(U1-Pad13) -> unconnected-(U1-D6-Pad13)
- U1 pad 14: Net-(U1-Pad14) -> unconnected-(U1-D7-Pad14)
- U1 pad 15: Net-(U1-Pad15) -> unconnected-(U1-D8-Pad15)
- U1 pad 3: Net-(U1-Pad3) -> unconnected-(U1-D4-Pad3)
- U1 pad 4: /TEMP -> /RELAY
- U1 pad 7: Net-(U1-Pad7) -> unconnected-(U1-Rx-Pad7)
- U1 pad 8: Net-(U1-Pad8) -> unconnected-(U1-Tx-Pad8)
- U1 pad 9: Net-(U1-Pad9) -> unconnected-(U1-Rst-Pad9)
Other:
- net class Default removed
